File: Kicad/Amstrad_PPC_Internal_CF_Lite.kicad_pcb (KiCad board)
At the start: 2 copper layers, 120 x 205 mm, 36 parts, among them J1 Amstrad_PPC_ISA_Connector_B, J2 Amstrad_PPC_ISA_Connector_A, J3 CONN_CF_CARD, J4 Conn_01x02, SW1 Switch_DIP_4_Positions, SW2 Switch_DIP_8_Positions, U1 74HCT244, U2 74HCT244, U3 74HCT688, U4 74LS32, U5 74HCT04, U6 74HCT688, U7 28C256

Commit message: Refinements to PCB
Parts:
- D1: footprint My_Components:LED_5mm -> Connector_PinHeader_2.54mm:PinHeader_1x02_P2.54mm_Vertical
- R1, R2, R3, R4, R5, R6, R7, R8: footprint Resistor_THT:R_Axial_DIN0207_L6.3mm_D2.5mm_P2.54mm_Vertical -> Resistor_THT:R_Axial_DIN0207_L6.3mm_D2.5mm_P7.62mm_Horizontal
- moved J4 60.4 mm to (85.6, 101.3)
- moved D1 18.2 mm to (110.5, 47.0), turned to 90 degrees
- moved R7 9.23 mm to (108.0, 39.6)
- moved R8 6.73 mm to (108.0, 31.5)
- moved SW1 6.03 mm to (85.1, 114.3)
- moved C3 5.12 mm to (89.7, 183.9), turned to -90 degrees
- moved C7 4.76 mm to (72.4, 84.1), turned to 180 degrees
- moved R5 3.06 mm to (40.1, 37.8)
- moved R4 3.06 mm to (40.1, 30.7)
- moved R6 3.06 mm to (40.1, 45.5)
- moved C8 1.27 mm to (50.6, 203.2)
- moved C6 0.94 mm to (62.5, 110.2)
- moved U4 0.57 mm to (66.3, 89.4)
- moved R3 0.49 mm to (78.0, 132.1)
- moved C2 0.44 mm to (59.5, 223.8)
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Connections:
- J3 pad : GND -> (no net)
Routing:
- net Net-(J4-Pin_1): track 7.62 -> 82.3 mm
- net Net-(J4-Pin_2): track 101.3 -> 37.5 mm, vias 1 -> 0
- net GND: track 753.6 -> 702.2 mm, vias 27 -> 20
- net /AEN: track 88.1 -> 53.7 mm, vias 2 -> 1
- net /~{IOR}: track 141.7 -> 112.3 mm
- net /B_A02: track 194.0 -> 166.1 mm, vias 4 -> 1
- net /A09: track 57.7 -> 82.3 mm
- net /~{CF_RESET}: track 94.0 -> 117.8 mm, vias 1 -> 3
- net Net-(D1-K): track 124.8 -> 103.4 mm
- net VCC: track 536.0 -> 554.3 mm
- net /B_A01: track 158.6 -> 176.0 mm, vias 3 -> 2
- net /D1: track 159.0 -> 145.6 mm
- net /D6: track 166.1 -> 176.8 mm, vias 3 -> 2
- net /~{MEMR}: track 123.4 -> 113.4 mm, vias 4 -> 1
- net /A12: track 42.2 -> 51.0 mm
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